File: prototipus.kicad_sch (KiCad schematic)
At the start: 9 parts, among them J1 Conn_01x04, J2 Conn_01x02, U1 ESP32-DEVKITC-32U

Commit message: docs: add schematic images, pdfs and update readme
Other:
- note added: "microSD module"
- note removed: "microSD"
Changed lines of the file:
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@@
 		)
 	)
-	(text "microSD"
+	(text "microSD module"
 		(exclude_from_sim no)
 		(at 157.988 41.656 0)
